File: kicad/hm-env-sensor.sch (KiCad schematic (older format))
At the start: 62 parts, among them Q1 Q12MHz/20pF/10ppm/4P/3.2x2.5mm, Q2 BC817-40(SOT23), Q3 BC817-40(SOT23), U1 BL4054B-42TPRN(SOT23-5), U2 CH340T(SSOP20W), U3 SY8089AAAC(SOT23-5), U4 BAT54C(SOT23-3), U5 ESP-WROOM-32, U6 BQ27441-G1, U7 BME280

Commit message: Rev B updates
Parts:
- removed BAT1: DW02S, OLIMEX_Connectors-FP:LIPO_BAT-CON2DW02R, symbol hm-env-sensor-rescue:BAT_CON-OLIMEX_Connectors-ESP32-DevKit-Lipo_Rev_A1-rescue
- removed C1, C6, C7: 47uF/6.3V/20%/X5R/C0805, OLIMEX_RLC-FP:C_0805_5MIL_DWS, symbol hm-env-sensor-rescue:C-OLIMEX_RCL-ESP32-DevKit-Lipo_Rev_A1-rescue
- removed C10, C11: 100nF/50V/20%/Y5V/C0603, OLIMEX_RLC-FP:C_0603_5MIL_DWS, symbol hm-env-sensor-rescue:0.1UF-25V-5%(0603)-SparkFun_BME280_Breakout_v10-eagle-impo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
- removed C2, C3: 27pF/50V/5%/C0G/C0603, OLIMEX_RLC-FP:C_0603_5MIL_DWS, symbol hm-env-sensor-rescue:C-OLIMEX_RCL-ESP32-DevKit-Lipo_Rev_A1-rescue
- removed C4: 22uF/6.3V/20%/X5R/C0603, OLIMEX_RLC-FP:C_0603_5MIL_DWS, symbol hm-env-sensor-rescue:C-OLIMEX_RCL-ESP32-DevKit-Lipo_Rev_A1-rescue
- removed C5: 100nF/50V/20%/Y5V/C0603, OLIMEX_RLC-FP:C_0603_5MIL_DWS, symbol hm-env-sensor-rescue:C-OLIMEX_RCL-ESP32-DevKit-Lipo_Rev_A1-rescue
- removed C8: 1.0uF/16V/10%/Y5V/C0603, OLIMEX_RLC-FP:C_0603_5MIL_DWS, symbol hm-env-sensor-rescue:1.0UF-16V-10%(0603)-sparkfun-battery-babysitter-eagle-impo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
- removed C9: 0.47uF/50V/20%/Y5V/C0603, OLIMEX_RLC-FP:C_0603_5MIL_DWS, symbol hm-env-sensor-rescue:CAP0603-CAP-sparkfun-battery-babysitter-eagle-import-esp32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
- removed D1, D2: 1N5822/SS34/SMA, OLIMEX_Diodes-FP:SMA-KA, symbol hm-env-sensor-rescue:D_Schottky-OLIMEX_Diodes-ESP32-DevKit-Lipo_Rev_A1-rescue
- removed D_Com1, GND1: TESTPAD, OLIMEX_Other-FP:TESTPAD_40-ROUND, symbol hm-env-sensor-rescue:TESTPAD-OLIMEX_OTHER-ESP32-DevKit-Lipo_Rev_A1-rescue
- removed EXT1, EXT2: HN1x19, OLIMEX_Connectors-FP:HN1x19, symbol hm-env-sensor-rescue:CON19-OLIMEX_Connectors-ESP32-DevKit-Lipo_Rev_A1-rescue
- removed FET1: WPM2015-3/TR, OLIMEX_Transistors-FP:SOT23, symbol hm-env-sensor-rescue:P-MOS+DIOD-OLIMEX_Transistors-ESP32-DevKit-Lipo_Rev_A1-res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
- removed L1: 2.2uH/1.5A/DCR<0.1R/CD32, OLIMEX_RLC-FP:CD32, symbol hm-env-sensor-rescue:L-OLIMEX_RCL-ESP32-DevKit-Lipo_Rev_A1-rescue
- removed PWRLED1: LED/RED/0603, OLIMEX_LEDs-FP:LED_0603_KA, symbol hm-env-sensor-rescue:LED-OLIMEX_Diodes-ESP32-DevKit-Lipo_Rev_A1-rescue
- removed Q1: Q12MHz/20pF/10ppm/4P/3.2x2.5mm, OLIMEX_Crystal-FP:TSX-3.2x2.5mm_GND(3), symbol hm-env-sensor-rescue:Crystal_GND-OLIMEX_Devices-ESP32-DevKit-Lipo_Rev_A1-rescue
- removed Q2, Q3: BC817-40(SOT23), OLIMEX_Transistors-FP:SOT23, symbol hm-env-sensor-rescue:Q_NPN_BEC-OLIMEX_Transistors-ESP32-DevKit-Lipo_Rev_A1-resc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
- removed R1: 10k/R0603, OLIMEX_RLC-FP:R_0603_5MIL_DWS, symbol hm-env-sensor-rescue:R-OLIMEX_RCL-ESP32-DevKit-Lipo_Rev_A1-rescue
- removed R10, R6, R7: 220R/R0603, OLIMEX_RLC-FP:R_0603_5MIL_DWS, symbol hm-env-sensor-rescue:R-OLIMEX_RCL-ESP32-DevKit-Lipo_Rev_A1-rescue
- removed R11: 4.99k/1%/R0603, OLIMEX_RLC-FP:R_0603_5MIL_DWS, symbol hm-env-sensor-rescue:R-OLIMEX_RCL-ESP32-DevKit-Lipo_Rev_A1-rescue
- removed R12: 1.1k/1%/R0603, OLIMEX_RLC-FP:R_0603_5MIL_DWS, symbol hm-env-sensor-rescue:R-OLIMEX_RCL-ESP32-DevKit-Lipo_Rev_A1-rescue
- removed R15: 0.01/1%/R1206, OLIMEX_RLC-FP:R_1206_5MIL_DWS, symbol hm-env-sensor-rescue:RESISTOR1206-sparkfun-battery-babysitter-eagle-import-esp3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
- removed R17, R19, R20, R21: 4.7k/R0603, OLIMEX_RLC-FP:R_0603_5MIL_DWS, symbol hm-env-sensor-rescue:4.7KOHM-1_10W-1%(0603)-SparkFun_BME280_Breakout_v10-eagle-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
- removed R2, R3, R4: 2.2k/R0603, OLIMEX_RLC-FP:R_0603_5MIL_DWS, symbol hm-env-sensor-rescue:R-OLIMEX_RCL-ESP32-DevKit-Lipo_Rev_A1-rescue
- removed R5: NA/R0603, OLIMEX_RLC-FP:R_0603_5MIL_DWS, symbol hm-env-sensor-rescue:R-OLIMEX_RCL-ESP32-DevKit-Lipo_Rev_A1-rescue
- removed R8, R9: 1k/R0603, OLIMEX_RLC-FP:R_0603_5MIL_DWS, symbol hm-env-sensor-rescue:R-OLIMEX_RCL-ESP32-DevKit-Lipo_Rev_A1-rescue
- removed RST3: IT-1185AU2-160G-G-TR, OLIMEX_Buttons-FP:IT1185AU2_V2, symbol hm-env-sensor-rescue:SIDE_WTCM-TR(3x4)-OLIMEX_Buttons-ESP32-DevKit-Lipo_Rev_A1-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
- removed U1: BL4054B-42TPRN(SOT23-5), OLIMEX_IC-FP:SOT-23-5, symbol hm-env-sensor-rescue:BL4054B-42TPRN(SOT23-5)-OLIMEX_IC-ESP32-DevKit-Lipo_Rev_A1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
- removed U2: CH340T(SSOP20W), OLIMEX_IC-FP:SSOP-20W, symbol hm-env-sensor-rescue:CH340T(SSOP20W)-OLIMEX_IC-ESP32-DevKit-Lipo_Rev_A1-rescue
- removed U3: SY8089AAAC(SOT23-5), OLIMEX_Regulators-FP:SOT-23-5, symbol hm-env-sensor-rescue:SY8009AAAC(SOT23-5)-OLIMEX_IC-ESP32-DevKit-Lipo_Rev_A1-res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
- removed U4: BAT54C(SOT23-3), OLIMEX_Diodes-FP:SOT23-3, symbol hm-env-sensor-rescue:BAT54C(SOT23-3)-OLIMEX_Diodes-ESP32-DevKit-Lipo_Rev_A1-res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
- removed U6: BQ27441-G1, sparkfun-battery-babysitter:PDSO-N12, symbol hm-env-sensor-rescue:BQ27441-G1-sparkfun-battery-babysitter-eagle-import-esp32-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
- removed U7: BME280, SparkFun_BME280_Breakout_v10:BME280_LGA, symbol hm-env-sensor-rescue:BME280-SparkFun_BME280_Breakout_v10-eagle-import-ESP32-Dev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
- removed USB-UART1: MISB-SWMM-5B-LF(USB_MICRO), OLIMEX_Connectors-FP:USB-MICRO_MISB-SWMM-5B_LF, symbol hm-env-sensor-rescue:USB-MINI-OLIMEX_Connectors-ESP32-DevKit-Lipo_Rev_A1-rescue
- added C22: 10uF/6.3V/X7R/C0603, OLIMEX_RLC-FP:C_0603_5MIL_DWS, symbol Device:C
- added FID1, FID2: Fiducial, OLIMEX_Other-FP:Fiducial1x3, symbol hm-env-sensor-rescue:Fiducial-OLIMEX_OTHER-ESP32-DevKit-Lipo_Rev_A1-rescue
- added J1: Conn_02x06_Odd_Even, Connector_PinHeader_2.54mm:PinHeader_2x06_P2.54mm_Vertical, symbol Connector_Generic:Conn_02x06_Odd_Even
- added R1: 330/R0603, OLIMEX_RLC-FP:R_0603_5MIL_DWS, symbol hm-env-sensor-rescue:4.7KOHM-1_10W-1%(0603)-SparkFun_BME280_Breakout_v10-eagle-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
- added R15: 4.7k/R0603, OLIMEX_RLC-FP:R_0603_5MIL_DWS, symbol hm-env-sensor-rescue:4.7KOHM-1_10W-1%(0603)-SparkFun_BME280_Breakout_v10-eagle-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
- R16: value 10k/R0603 -> 4.7k/R0603
Connections:
- net +3V3: now also R16.2, C22.1, J1.4 (Pin_4), R15.2
- net +5V: now also J1.2 (Pin_2); no longer CHARGING1.2 (A)
- net GND: now also C22.2, J1.6 (Pin_6), R1.1; no longer R16.1
- net GPI34: now also J1.12 (Pin_12)
- net GPI35: now also J1.10 (Pin_10)
- net GPIO22: now also CHARGING1.2 (A)
- net GPIO23: now also J1.5 (Pin_5)
- net GPIO27: now also J1.7 (Pin_7)
- net GPIO32: now also J1.9 (Pin_9), R15.1
- net GPIO33: now also R16.1, J1.11 (Pin_11)
- net GPIO4: now also J1.1 (Pin_1)
- net GPIO5: now also J1.3 (Pin_3)
- net at CHARGING1.1 (K): now also R1.2
- net GPI36/SENSOR_VP renamed GPI36
- net GPI39/SENSOR_VN renamed GPI39
- net GPI39: now also J1.8 (Pin_8)
- net GPIO1/U0TXD renamed GPIO1
- net GPIO10/SD_DATA3: no longer names the net of U5.18 (GPIO10/SD_DATA3/SPIWP/HS1_DATA3/U1TXD)
- net GPIO11/SD_CMD: no longer names the net of U5.19 (GPIO11/SD_CMD/SPICS0/HS1_CMD/U1RTS)
- net GPIO12: no longer names the net of U5.14 (GPIO12/ADC2_CH5/TOUCH5/RTC_GPIO15/MTDI/HSPIQ/HS2_DATA2/SD_DATA2/EMAC_TXD3)
- net GPIO3/U0RXD renamed GPIO3
- net GPIO6/SD_CLK: no longer names the net of U5.20 (GPIO6/SD_CLK/SPICLK/HS1_CLK/U1CTS)
- net GPIO7/SD_DATA0: no longer names the net of U5.21 (GPIO7/SD_DATA0/SPIQ/HS1_DATA0/U2RTS)
- net GPIO8/SD_DATA1: no longer names the net of U5.22 (GPIO8/SD_DATA1/SPID/HS1_DATA1/U2CTS)
- net GPIO9/SD_DATA2: no longer names the net of U5.17 (GPIO9/SD_DATA2/SPIHD/HS1_DATA2/U1RXD)
- no-connect marks 6 -> 7
Other:
- note added: "Power\n"
- note added: "Sensors"
- note removed: "0"
- note removed: "1"
- note removed: "Auto program\n"
- note removed: "BATTERY_IN goes to \nthe battery connector\nBAT1 pin 1 (+)"
- note removed: "BME280"
- note removed: "BQ27441-G1 Fuel Gauge"
- note removed: "DTR RTS->EN IO0"
- note removed: "Fuel Gauge"
- note removed: "I2C ADDR: 0x55"
- note removed: "I2C ADDR: 0x77 or 0x76"
- note removed: "IBAT = 1000/Rprog = 455mA"
- note removed: "LiPo Charger"
- note removed: "PENDING"
- note removed: "Power Supply"
- note removed: "Ra"
- note removed: "Rb"
- note removed: "Rprog"
- note removed: "SDO to ground \nwill set default I2C address"
- note removed: "The BQ27441-G1\ngoes between here"
- note removed: "Two reset button, we keep the original \nplacement of the reset button, and \nwe add a reset button that will be \naccessible via the ventilation holes in the enclosure."
- note removed: "USB to UART"
- note removed: "VDD is 1.8V\ngenerated internally"
- note removed: "Vout=0.6*(1+Ra/Rb)"
- moved on the sheet: D4, D6, FID3, R13, R14, R22, R24, R26, RST1, RST2, U5
